File: pcb/main_board/NixieSTM32.kicad_pcb (KiCad board)
At the start: 4 copper layers, 108 x 48.5 mm, 54 parts, among them J1 Conn_ARM_SWD_6, J2 Conn_02x06_Odd_Even, J3 Conn_02x06_Odd_Even, J4 Conn_02x06_Odd_Even, J5 Conn_02x06_Odd_Even, M1 74141DIP16, M2 74141DIP16, M3 74141DIP16, M4 74141DIP16, Q1 FQU11P06TU, SW1 SW_SPDT, U1 STM32L010K4T6, U2 MAX6817, U3 TPS7A05SOT23, U4 LT3470ITS8PBF, U5 NCH8200HV, Y1 32.768kHz

Commit message: Adding images and updating README.
Connections:
- net +9V renamed SHDN_LT3470
- net VDDA renamed Net-(U1-VDDA)
